Commit message: [ffb] Make WheelFR_link the parent of base_footprint

File: urdf/pepper_ffb.urdf (robot description, URDF)
Before this commit: robot JulietteY20MP, 83 links, 82 joints
Joints:
- joint base_footprint_joint: parent Tibia -> WheelFR_link

Commit message: Change Pepper FFB kinematic tree
- Make wheel the root link
- Add VREP import of the model

File: urdf/pepper_ffb.urdf (robot description, URDF)
Before this commit: robot JulietteY20MP, 83 links, 82 joints
Joints:
- joint HipPitch: child Pelvis -> Hip; origin xyz=0 0 -0.079 rpy=0 0 0 -> xyz=0 0 0.079 rpy=0 0 0; parent Hip -> Pelvis
- joint HipRoll: child Hip -> torso; origin xyz=2e-05 0 -0.139 rpy=0 0 0 -> xyz=2e-05 0 0.139 rpy=0 0 0; parent torso -> Hip
- joint KneePitch: child Tibia -> Pelvis; origin xyz=0 0 -0.268 rpy=0 0 0 -> xyz=0 0 0.268 rpy=0 0 0; parent Pelvis -> Tibia
- joint Rot_Z: child WheelFL_link -> WheelB_link; origin xyz=0.0 0. 0. rpy=0 0 0 -> xyz=0 0 0 rpy=0 0 0; parent Tibia -> WheelFR_link
- joint Trans_X: child WheelB_link -> WheelFL_link; parent WheelFL_link -> WheelB_link
- joint Trans_Y: axis 00 1.0 0 -> 0 1.0 0; child WheelFR_link -> Tibia; origin xyz=0 0 0 rpy=0 0 0 -> xyz=0.0 0. 0. rpy=0 0 0; parent WheelB_link -> WheelFL_link
- joint base_footprint_joint: child base_footprint -> WheelFR_link; origin xyz=0 0 -0.334 rpy=0 0 0 -> xyz=0 0 0.334 rpy=0 0 0; parent WheelFR_link -> base_footprint
- joint base_link_fixedjoint: child torso -> base_footprint

Commit message: Corrected FFB VREP model

File: urdf/pepper_ffb.urdf (robot description, URDF)
Before this commit: robot JulietteY20MP, 83 links, 82 joints
Joints:
- joint Rot_Z: child WheelB_link -> Tibia; origin xyz=0 0 0 rpy=0 0 0 -> xyz=0.0 0. 0. rpy=0 0 0; parent WheelFR_link -> WheelFL_link
- joint Trans_Y: child Tibia -> WheelB_link; origin xyz=0.0 0. 0. rpy=0 0 0 -> xyz=0 0 0 rpy=0 0 0; parent WheelFL_link -> WheelFR_link
- joint base_footprint_joint: origin xyz=0 0 0.334 rpy=0 0 0 -> xyz=0 0 0 rpy=0 0 0

Commit message: Correct all axis on URDF and VREP behaviour

File: urdf/pepper_ffb.urdf (robot description, URDF)
Before this commit: robot JulietteY20MP, 83 links, 82 joints
Links:
- removed link BumperB_frame
- removed link BumperFL_frame
- removed link BumperFR_frame
- removed link CameraBottom_frame
- removed link CameraBottom_optical_frame
- removed link CameraDepth_frame
- removed link CameraDepth_optical_frame
- removed link CameraTop_frame
- removed link CameraTop_optical_frame
- removed link ChestButton_frame
- removed link HeadTouchFront_frame
- removed link HeadTouchMiddle_frame
- removed link HeadTouchRear_frame
- removed link ImuBaseAccelerometer_frame
- removed link ImuTorsoAccelerometer_frame
- removed link ImuTorsoGyrometer_frame
- removed link LHandTouchBack_frame
- removed link LSpeaker_frame
- removed link RHandTouchBack_frame
- removed link RSpeaker_frame
- removed link ShovelLaser_frame
- removed link SonarBack_frame
- removed link SonarFront_frame
- removed link SurroundingFrontLaser_device_frame
- removed link SurroundingFrontLaser_frame
- removed link SurroundingLeftLaser_device_frame
- removed link SurroundingLeftLaser_frame
- removed link SurroundingRightLaser_device_frame
- removed link SurroundingRightLaser_frame
- removed link Tablet_frame
- removed link VerticalLeftLaser_frame
- removed link VerticalRightLaser_frame
- link Tibia: geometry collision mesh filename=package://pepper_description/meshes/KneePitch_0.10.stl scale=0.1 0.1 0.1; collision mesh filename=package://pepper_description/meshes/WheelB_0.10.stl scale=0.1 0.1 0.1
Joints:
- removed joint AccelerometerBase_sensor_fixedjoint
- removed joint Accelerometer_sensor_fixedjoint
- removed joint Bumper/Back_sensor_fixedjoint
- removed joint Bumper/FrontLeft_sensor_fixedjoint
- removed joint Bumper/FrontRight_sensor_fixedjoint
- removed joint CameraBottom_optical_frame_fixedjoint
- removed joint CameraBottom_sensor_fixedjoint
- removed joint CameraDepth_optical_frame_fixedjoint
- removed joint CameraDepth_sensor_fixedjoint
- removed joint CameraTop_optical_frame_fixedjoint
- removed joint CameraTop_sensor_fixedjoint
- removed joint ChestBoard/Button_sensor_fixedjoint
- removed joint Gyrometer_sensor_fixedjoint
- removed joint Head/Touch/Front_sensor_fixedjoint
- removed joint Head/Touch/Middle_sensor_fixedjoint
- removed joint Head/Touch/Rear_sensor_fixedjoint
- removed joint LHand/Touch/Back_sensor_fixedjoint
- removed joint LaserSensor/Front_projected_sensor_fixedjoint
- removed joint LaserSensor/Front_sensor_fixedjoint
- removed joint LaserSensor/Left_projected_sensor_fixedjoint
- removed joint LaserSensor/Left_sensor_fixedjoint
- removed joint LaserSensor/Right_projected_sensor_fixedjoint
- removed joint LaserSensor/Right_sensor_fixedjoint
- removed joint LaserSensor/Shovel_sensor_fixedjoint
- removed joint LaserSensor/VerticalLeft_sensor_fixedjoint
- removed joint LaserSensor/VerticalRight_sensor_fixedjoint
- removed joint RHand/Touch/Back_sensor_fixedjoint
- removed joint Sonar/Back_sensor_fixedjoint
- removed joint Sonar/Front_sensor_fixedjoint
- removed joint SpeakerLeft_sensor_fixedjoint
- removed joint SpeakerRight_sensor_fixedjoint
- removed joint Tablet_sensor_fixedjoint
- joint HeadYaw: origin xyz=-0.038 0 0.1699 rpy=0 0 0 -> xyz=-0.038 0 0.3089 rpy=0 0 0
- joint HipPitch: origin xyz=0 0 0.079 rpy=0 0 0 -> xyz=0 0 0.268 rpy=0 0 0
- joint HipRoll: origin xyz=2e-05 0 0.139 rpy=0 0 0 -> xyz=0 0 0.079 rpy=0 0 0
- joint KneePitch: origin xyz=0 0 0.268 rpy=0 0 0 -> xyz=0 0 0 rpy=0 0 0
- joint LShoulderPitch: origin xyz=-0.057 0.14974 0.08682 rpy=0 0 0 -> xyz=-0.057 0.14974 0.22582 rpy=0 0 0
- joint RShoulderPitch: origin xyz=-0.057 -0.14974 0.08682 rpy=0 0 0 -> xyz=-0.057 -0.14974 0.22582 rpy=0 0 0
