Commit message: Removed finger/hand joints from simplified model files, edited surfaces

File: urdf/pepper_no_fingers.urdf (robot description, URDF)
Before this commit: robot JulietteY20MP, 23 links, 22 joints
Links:
- removed link l_gripper
- removed link r_gripper
Joints:
- removed joint LHand
- removed joint RHand
