Commit message: Use the packages' meshes

File: urdf/pepper.urdf (robot description, URDF)
Before this commit: robot JulietteY20MP, 83 links, 82 joints
Links:
- link Head: geometry collision mesh filename=package://pepper_description/meshes/HeadPitch_0.10.stl scale=0.1 0.1 0.1; visual mesh filename=package://pepper_description/meshes/HeadPitch.dae scale=0.1 0.1 0.1
- link Hip: geometry collision mesh filename=package://pepper_description/meshes/HipRoll_0.10.stl scale=0.1 0.1 0.1; visual mesh filename=package://pepper_description/meshes/HipRoll.dae scale=0.1 0.1 0.1
- link LBicep: geometry collision mesh filename=package://pepper_description/meshes/LShoulderRoll_0.10.stl scale=0.1 0.1 0.1; visual mesh filename=package://pepper_description/meshes/LShoulderRoll.dae scale=0.1 0.1 0.1
- link LElbow: geometry collision mesh filename=package://pepper_description/meshes/LElbowYaw_0.10.stl scale=0.1 0.1 0.1; visual mesh filename=package://pepper_description/meshes/LElbowYaw.dae scale=0.1 0.1 0.1
- link LFinger11_link: geometry collision mesh filename=package://pepper_description/meshes/LFinger11_0.10.stl scale=0.1 0.1 0.1; visual mesh filename=package://pepper_description/meshes/LFinger11.dae scale=0.1 0.1 0.1
- link LFinger12_link: geometry collision mesh filename=package://pepper_description/meshes/LFinger12_0.10.stl scale=0.1 0.1 0.1; visual mesh filename=package://pepper_description/meshes/LFinger12.dae scale=0.1 0.1 0.1
- link LFinger13_link: geometry collision mesh filename=package://pepper_description/meshes/LFinger13_0.10.stl scale=0.1 0.1 0.1; visual mesh filename=package://pepper_description/meshes/LFinger13.dae scale=0.1 0.1 0.1
- link LFinger21_link: geometry collision mesh filename=package://pepper_description/meshes/LFinger21_0.10.stl scale=0.1 0.1 0.1; visual mesh filename=package://pepper_description/meshes/LFinger21.dae scale=0.1 0.1 0.1
- link LFinger22_link: geometry collision mesh filename=package://pepper_description/meshes/LFinger22_0.10.stl scale=0.1 0.1 0.1; visual mesh filename=package://pepper_description/meshes/LFinger22.dae scale=0.1 0.1 0.1
- link LFinger23_link: geometry collision mesh filename=package://pepper_description/meshes/LFinger23_0.10.stl scale=0.1 0.1 0.1; visual mesh filename=package://pepper_description/meshes/LFinger23.dae scale=0.1 0.1 0.1
- link LFinger31_link: geometry collision mesh filename=package://pepper_description/meshes/LFinger31_0.10.stl scale=0.1 0.1 0.1; visual mesh filename=package://pepper_description/meshes/LFinger31.dae scale=0.1 0.1 0.1
- link LFinger32_link: geometry collision mesh filename=package://pepper_description/meshes/LFinger32_0.10.stl scale=0.1 0.1 0.1; visual mesh filename=package://pepper_description/meshes/LFinger32.dae scale=0.1 0.1 0.1
- link LFinger33_link: geometry collision mesh filename=package://pepper_description/meshes/LFinger33_0.10.stl scale=0.1 0.1 0.1; visual mesh filename=package://pepper_description/meshes/LFinger33.dae scale=0.1 0.1 0.1
- link LFinger41_link: geometry collision mesh filename=package://pepper_description/meshes/LFinger41_0.10.stl scale=0.1 0.1 0.1; visual mesh filename=package://pepper_description/meshes/LFinger41.dae scale=0.1 0.1 0.1
- link LFinger42_link: geometry collision mesh filename=package://pepper_description/meshes/LFinger42_0.10.stl scale=0.1 0.1 0.1; visual mesh filename=package://pepper_description/meshes/LFinger42.dae scale=0.1 0.1 0.1
- link LFinger43_link: geometry collision mesh filename=package://pepper_description/meshes/LFinger43_0.10.stl scale=0.1 0.1 0.1; visual mesh filename=package://pepper_description/meshes/LFinger43.dae scale=0.1 0.1 0.1
- link LForeArm: geometry collision mesh filename=package://pepper_description/meshes/LElbowRoll_0.10.stl scale=0.1 0.1 0.1; visual mesh filename=package://pepper_description/meshes/LElbowRoll.dae scale=0.1 0.1 0.1
- link LShoulder: geometry collision mesh filename=package://pepper_description/meshes/LShoulderPitch_0.10.stl scale=0.1 0.1 0.1; visual mesh filename=package://pepper_description/meshes/LShoulderPitch.dae scale=0.1 0.1 0.1
- link LThumb1_link: geometry collision mesh filename=package://pepper_description/meshes/LThumb1_0.10.stl scale=0.1 0.1 0.1; visual mesh filename=package://pepper_description/meshes/LThumb1.dae scale=0.1 0.1 0.1
- link LThumb2_link: geometry collision mesh filename=package://pepper_description/meshes/LThumb2_0.10.stl scale=0.1 0.1 0.1; visual mesh filename=package://pepper_description/meshes/LThumb2.dae scale=0.1 0.1 0.1
- link Neck: geometry collision mesh filename=package://pepper_description/meshes/HeadYaw_0.10.stl scale=0.1 0.1 0.1; visual mesh filename=package://pepper_description/meshes/HeadYaw.dae scale=0.1 0.1 0.1
- link Pelvis: geometry collision mesh filename=package://pepper_description/meshes/HipPitch_0.10.stl scale=0.1 0.1 0.1; visual mesh filename=package://pepper_description/meshes/HipPitch.dae scale=0.1 0.1 0.1
- link RBicep: geometry collision mesh filename=package://pepper_description/meshes/RShoulderRoll_0.10.stl scale=0.1 0.1 0.1; visual mesh filename=package://pepper_description/meshes/RShoulderRoll.dae scale=0.1 0.1 0.1
- link RElbow: geometry collision mesh filename=package://pepper_description/meshes/RElbowYaw_0.10.stl scale=0.1 0.1 0.1; visual mesh filename=package://pepper_description/meshes/RElbowYaw.dae scale=0.1 0.1 0.1
- link RFinger11_link: geometry collision mesh filename=package://pepper_description/meshes/RFinger11_0.10.stl scale=0.1 0.1 0.1; visual mesh filename=package://pepper_description/meshes/RFinger11.dae scale=0.1 0.1 0.1
- link RFinger12_link: geometry collision mesh filename=package://pepper_description/meshes/RFinger12_0.10.stl scale=0.1 0.1 0.1; visual mesh filename=package://pepper_description/meshes/RFinger12.dae scale=0.1 0.1 0.1
- link RFinger13_link: geometry collision mesh filename=package://pepper_description/meshes/RFinger13_0.10.stl scale=0.1 0.1 0.1; visual mesh filename=package://pepper_description/meshes/RFinger13.dae scale=0.1 0.1 0.1
- link RFinger21_link: geometry collision mesh filename=package://pepper_description/meshes/RFinger21_0.10.stl scale=0.1 0.1 0.1; visual mesh filename=package://pepper_description/meshes/RFinger21.dae scale=0.1 0.1 0.1
- link RFinger22_link: geometry collision mesh filename=package://pepper_description/meshes/RFinger22_0.10.stl scale=0.1 0.1 0.1; visual mesh filename=package://pepper_description/meshes/RFinger22.dae scale=0.1 0.1 0.1
- link RFinger23_link: geometry collision mesh filename=package://pepper_description/meshes/RFinger23_0.10.stl scale=0.1 0.1 0.1; visual mesh filename=package://pepper_description/meshes/RFinger23.dae scale=0.1 0.1 0.1
- link RFinger31_link: geometry collision mesh filename=package://pepper_description/meshes/RFinger31_0.10.stl scale=0.1 0.1 0.1; visual mesh filename=package://pepper_description/meshes/RFinger31.dae scale=0.1 0.1 0.1
- link RFinger32_link: geometry collision mesh filename=package://pepper_description/meshes/RFinger32_0.10.stl scale=0.1 0.1 0.1; visual mesh filename=package://pepper_description/meshes/RFinger32.dae scale=0.1 0.1 0.1
- link RFinger33_link: geometry collision mesh filename=package://pepper_description/meshes/RFinger33_0.10.stl scale=0.1 0.1 0.1; visual mesh filename=package://pepper_description/meshes/RFinger33.dae scale=0.1 0.1 0.1
- link RFinger41_link: geometry collision mesh filename=package://pepper_description/meshes/RFinger41_0.10.stl scale=0.1 0.1 0.1; visual mesh filename=package://pepper_description/meshes/RFinger41.dae scale=0.1 0.1 0.1
- link RFinger42_link: geometry collision mesh filename=package://pepper_description/meshes/RFinger42_0.10.stl scale=0.1 0.1 0.1; visual mesh filename=package://pepper_description/meshes/RFinger42.dae scale=0.1 0.1 0.1
- link RFinger43_link: geometry collision mesh filename=package://pepper_description/meshes/RFinger43_0.10.stl scale=0.1 0.1 0.1; visual mesh filename=package://pepper_description/meshes/RFinger43.dae scale=0.1 0.1 0.1
- link RForeArm: geometry collision mesh filename=package://pepper_description/meshes/RElbowRoll_0.10.stl scale=0.1 0.1 0.1; visual mesh filename=package://pepper_description/meshes/RElbowRoll.dae scale=0.1 0.1 0.1
- link RShoulder: geometry collision mesh filename=package://pepper_description/meshes/RShoulderPitch_0.10.stl scale=0.1 0.1 0.1; visual mesh filename=package://pepper_description/meshes/RShoulderPitch.dae scale=0.1 0.1 0.1
- link RThumb1_link: geometry collision mesh filename=package://pepper_description/meshes/RThumb1_0.10.stl scale=0.1 0.1 0.1; visual mesh filename=package://pepper_description/meshes/RThumb1.dae scale=0.1 0.1 0.1
- link RThumb2_link: geometry collision mesh filename=package://pepper_description/meshes/RThumb2_0.10.stl scale=0.1 0.1 0.1; visual mesh filename=package://pepper_description/meshes/RThumb2.dae scale=0.1 0.1 0.1
- link Tibia: geometry collision mesh filename=package://pepper_description/meshes/KneePitch_0.10.stl scale=0.1 0.1 0.1; visual mesh filename=package://pepper_description/meshes/KneePitch.dae scale=0.1 0.1 0.1
- link WheelB_link: geometry collision mesh filename=package://pepper_description/meshes/WheelB_0.10.stl scale=0.1 0.1 0.1; visual mesh filename=package://pepper_description/meshes/WheelB.dae scale=0.1 0.1 0.1
- link WheelFL_link: geometry collision mesh filename=package://pepper_description/meshes/WheelFL_0.10.stl scale=0.1 0.1 0.1; visual mesh filename=package://pepper_description/meshes/WheelFL.dae scale=0.1 0.1 0.1
- link WheelFR_link: geometry collision mesh filename=package://pepper_description/meshes/WheelFR_0.10.stl scale=0.1 0.1 0.1; visual mesh filename=package://pepper_description/meshes/WheelFR.dae scale=0.1 0.1 0.1
- link l_wrist: geometry collision mesh filename=package://pepper_description/meshes/LWristYaw_0.10.stl scale=0.1 0.1 0.1; visual mesh filename=package://pepper_description/meshes/LWristYaw.dae scale=0.1 0.1 0.1
- link r_wrist: geometry collision mesh filename=package://pepper_description/meshes/RWristYaw_0.10.stl scale=0.1 0.1 0.1; visual mesh filename=package://pepper_description/meshes/RWristYaw.dae scale=0.1 0.1 0.1
- link torso: geometry collision mesh filename=package://pepper_description/meshes/Torso_0.10.stl scale=0.1 0.1 0.1; visual mesh filename=package://pepper_description/meshes/Torso.dae scale=0.1 0.1 0.1

Commit message: Updated URDF: some inertia parameters from SBR, changed kinematic tree structure (base_link as root). Cleanup old files

File: urdf/pepper.urdf (robot description, URDF)
Before this commit: robot JulietteY20MP, 83 links, 82 joints
Links:
- removed link base_footprint
- added link HipOffset
- added link l_grasp_frame
- added link r_grasp_frame
Joints:
- removed joint base_footprint_joint
- removed joint base_link_fixedjoint
- added joint LGrasp: type fixed, parent l_wrist, child l_grasp_frame, origin xyz=0.070 0 0 rpy=3.1415 0 1.5707
- added joint RGrasp: type fixed, parent r_wrist, child r_grasp_frame, origin xyz=0.070 0 0 rpy=3.1415 0 1.5707
- added joint base_joint: type fixed, parent base_link, child Tibia, origin xyz=0 0 0.334 rpy=0 0 0
- added joint hip_fixed: type fixed, parent HipOffset, child torso, origin xyz=0 0 0.139 rpy=0 0 0
- joint HipPitch: axis 0 1.0 0 -> 0 -1.0 0; child Pelvis -> Hip; origin xyz=0 0 -0.079 rpy=0 0 0 -> xyz=0 0 0.268 rpy=0 0 0; parent Hip -> Pelvis
- joint HipRoll: axis 1.0 0 0 -> -1.0 0 0; child Hip -> HipOffset; origin xyz=2e-05 0 -0.139 rpy=0 0 0 -> xyz=-2e-05 0 0.079 rpy=0 0 0; parent torso -> Hip
- joint KneePitch: axis 0 1.0 0 -> 0 -1.0 0; child Tibia -> Pelvis; origin xyz=0 0 -0.268 rpy=0 0 0 -> xyz=0 0 0 rpy=0 0 0; parent Pelvis -> Tibia
- joint LFinger11: limit (none) -> lower=0 upper=0.86 effort=1 velocity=1; type continuous -> revolute
- joint LFinger12: limit (none) -> lower=0 upper=0.86 effort=1 velocity=1; type continuous -> revolute
- joint LFinger13: limit (none) -> lower=0 upper=0.86 effort=1 velocity=1; type continuous -> revolute
- joint LFinger21: limit (none) -> lower=0 upper=0.86 effort=1 velocity=1; type continuous -> revolute
- joint LFinger22: limit (none) -> lower=0 upper=0.86 effort=1 velocity=1; type continuous -> revolute
- joint LFinger23: limit (none) -> lower=0 upper=0.86 effort=1 velocity=1; type continuous -> revolute
- joint LFinger31: limit (none) -> lower=0 upper=0.86 effort=1 velocity=1; type continuous -> revolute
- joint LFinger32: limit (none) -> lower=0 upper=0.86 effort=1 velocity=1; type continuous -> revolute
- joint LFinger33: limit (none) -> lower=0 upper=0.86 effort=1 velocity=1; type continuous -> revolute
- joint LFinger41: limit (none) -> lower=0 upper=0.86 effort=1 velocity=1; type continuous -> revolute
- joint LFinger42: limit (none) -> lower=0 upper=0.86 effort=1 velocity=1; type continuous -> revolute
- joint LFinger43: limit (none) -> lower=0 upper=0.86 effort=1 velocity=1; type continuous -> revolute
- joint LThumb1: limit (none) -> lower=0 upper=0.86 effort=1 velocity=1; type continuous -> revolute
- joint LThumb2: limit (none) -> lower=0 upper=0.86 effort=1 velocity=1; type continuous -> revolute
- joint RFinger11: limit (none) -> lower=0 upper=0.86 effort=1 velocity=1; type continuous -> revolute
- joint RFinger12: limit (none) -> lower=0 upper=0.86 effort=1 velocity=1; type continuous -> revolute
- joint RFinger13: limit (none) -> lower=0 upper=0.86 effort=1 velocity=1; type continuous -> revolute
- joint RFinger21: limit (none) -> lower=0 upper=0.86 effort=1 velocity=1; type continuous -> revolute
- joint RFinger22: limit (none) -> lower=0 upper=0.86 effort=1 velocity=1; type continuous -> revolute
- joint RFinger23: limit (none) -> lower=0 upper=0.86 effort=1 velocity=1; type continuous -> revolute
- joint RFinger31: limit (none) -> lower=0 upper=0.86 effort=1 velocity=1; type continuous -> revolute
- joint RFinger32: limit (none) -> lower=0 upper=0.86 effort=1 velocity=1; type continuous -> revolute
- joint RFinger33: limit (none) -> lower=0 upper=0.86 effort=1 velocity=1; type continuous -> revolute
- joint RFinger41: limit (none) -> lower=0 upper=0.86 effort=1 velocity=1; type continuous -> revolute
- joint RFinger42: limit (none) -> lower=0 upper=0.86 effort=1 velocity=1; type continuous -> revolute
- joint RFinger43: limit (none) -> lower=0 upper=0.86 effort=1 velocity=1; type continuous -> revolute
- joint RThumb1: limit (none) -> lower=0 upper=0.86 effort=1 velocity=1; type continuous -> revolute
- joint RThumb2: limit (none) -> lower=0 upper=0.86 effort=1 velocity=1; type continuous -> revolute
- joint WheelB: type continuous -> fixed
- joint WheelFL: type continuous -> fixed
- joint WheelFR: type continuous -> fixed
