Commit message: Simplified FFB model, mobile base and fixed base models are now of the same general form

File: urdf/pepper.urdf (robot description, URDF)
Before this commit: robot JulietteY20MP, 85 links, 84 joints
Links:
- removed link BumperB_frame
- removed link BumperFL_frame
- removed link BumperFR_frame
- removed link CameraBottom_frame
- removed link CameraBottom_optical_frame
- removed link CameraDepth_frame
- removed link CameraDepth_optical_frame
- removed link ChestButton_frame
- removed link HeadTouchFront_frame
- removed link HeadTouchMiddle_frame
- removed link HeadTouchRear_frame
- removed link HipOffset
- removed link ImuBaseAccelerometer_frame
- removed link ImuTorsoAccelerometer_frame
- removed link ImuTorsoGyrometer_frame
- removed link LHandTouchBack_frame
- removed link LSpeaker_frame
- removed link RHandTouchBack_frame
- removed link RSpeaker_frame
- removed link ShovelLaser_frame
- removed link SonarBack_frame
- removed link SonarFront_frame
- removed link SurroundingFrontLaser_device_frame
- removed link SurroundingFrontLaser_frame
- removed link SurroundingLeftLaser_device_frame
- removed link SurroundingLeftLaser_frame
- removed link SurroundingRightLaser_device_frame
- removed link SurroundingRightLaser_frame
- removed link Tablet_frame
- removed link VerticalLeftLaser_frame
- removed link VerticalRightLaser_frame
- removed link l_grasp_frame
- removed link r_grasp_frame
Joints:
- removed joint AccelerometerBase_sensor_fixedjoint
- removed joint Accelerometer_sensor_fixedjoint
- removed joint Bumper/Back_sensor_fixedjoint
- removed joint Bumper/FrontLeft_sensor_fixedjoint
- removed joint Bumper/FrontRight_sensor_fixedjoint
- removed joint CameraBottom_optical_frame_fixedjoint
- removed joint CameraBottom_sensor_fixedjoint
- removed joint CameraDepth_optical_frame_fixedjoint
- removed joint CameraDepth_sensor_fixedjoint
- removed joint ChestBoard/Button_sensor_fixedjoint
- removed joint Gyrometer_sensor_fixedjoint
- removed joint Head/Touch/Front_sensor_fixedjoint
- removed joint Head/Touch/Middle_sensor_fixedjoint
- removed joint Head/Touch/Rear_sensor_fixedjoint
- removed joint LGrasp
- removed joint LHand/Touch/Back_sensor_fixedjoint
- removed joint LaserSensor/Front_projected_sensor_fixedjoint
- removed joint LaserSensor/Front_sensor_fixedjoint
- removed joint LaserSensor/Left_projected_sensor_fixedjoint
- removed joint LaserSensor/Left_sensor_fixedjoint
- removed joint LaserSensor/Right_projected_sensor_fixedjoint
- removed joint LaserSensor/Right_sensor_fixedjoint
- removed joint LaserSensor/Shovel_sensor_fixedjoint
- removed joint LaserSensor/VerticalLeft_sensor_fixedjoint
- removed joint LaserSensor/VerticalRight_sensor_fixedjoint
- removed joint RGrasp
- removed joint RHand/Touch/Back_sensor_fixedjoint
- removed joint Sonar/Back_sensor_fixedjoint
- removed joint Sonar/Front_sensor_fixedjoint
- removed joint SpeakerLeft_sensor_fixedjoint
- removed joint SpeakerRight_sensor_fixedjoint
- removed joint Tablet_sensor_fixedjoint
- removed joint base_joint
- removed joint hip_fixed
- added joint fixed_base: type fixed, parent base_link, child Tibia, origin xyz=0 0 0.334 rpy=0 0 0
- joint HeadYaw: origin xyz=-0.038 0 0.1699 rpy=0 0 0 -> xyz=-0.038 0 0.3089 rpy=0 0 0
- joint HipRoll: axis -1.0 0 0 -> 1.0 0 0; child HipOffset -> torso; origin xyz=-2e-05 0 0.079 rpy=0 0 0 -> xyz=0 0 0.079 rpy=0 0 0
- joint LFinger11: limit lower=0 upper=0.86 effort=1 velocity=1 -> (none); type revolute -> continuous
- joint LFinger12: limit lower=0 upper=0.86 effort=1 velocity=1 -> (none); type revolute -> continuous
- joint LFinger13: limit lower=0 upper=0.86 effort=1 velocity=1 -> (none); type revolute -> continuous
- joint LFinger21: limit lower=0 upper=0.86 effort=1 velocity=1 -> (none); type revolute -> continuous
- joint LFinger22: limit lower=0 upper=0.86 effort=1 velocity=1 -> (none); type revolute -> continuous
- joint LFinger23: limit lower=0 upper=0.86 effort=1 velocity=1 -> (none); type revolute -> continuous
- joint LFinger31: limit lower=0 upper=0.86 effort=1 velocity=1 -> (none); type revolute -> continuous
- joint LFinger32: limit lower=0 upper=0.86 effort=1 velocity=1 -> (none); type revolute -> continuous
- joint LFinger33: limit lower=0 upper=0.86 effort=1 velocity=1 -> (none); type revolute -> continuous
- joint LFinger41: limit lower=0 upper=0.86 effort=1 velocity=1 -> (none); type revolute -> continuous
- joint LFinger42: limit lower=0 upper=0.86 effort=1 velocity=1 -> (none); type revolute -> continuous
- joint LFinger43: limit lower=0 upper=0.86 effort=1 velocity=1 -> (none); type revolute -> continuous
- joint LShoulderPitch: origin xyz=-0.057 0.14974 0.08682 rpy=0 0 0 -> xyz=-0.057 0.14974 0.22582 rpy=0 0 0
- joint LThumb1: limit lower=0 upper=0.86 effort=1 velocity=1 -> (none); type revolute -> continuous
- joint LThumb2: limit lower=0 upper=0.86 effort=1 velocity=1 -> (none); type revolute -> continuous
- joint RFinger11: limit lower=0 upper=0.86 effort=1 velocity=1 -> (none); type revolute -> continuous
- joint RFinger12: limit lower=0 upper=0.86 effort=1 velocity=1 -> (none); type revolute -> continuous
- joint RFinger13: limit lower=0 upper=0.86 effort=1 velocity=1 -> (none); type revolute -> continuous
- joint RFinger21: limit lower=0 upper=0.86 effort=1 velocity=1 -> (none); type revolute -> continuous
- joint RFinger22: limit lower=0 upper=0.86 effort=1 velocity=1 -> (none); type revolute -> continuous
- joint RFinger23: limit lower=0 upper=0.86 effort=1 velocity=1 -> (none); type revolute -> continuous
- joint RFinger31: limit lower=0 upper=0.86 effort=1 velocity=1 -> (none); type revolute -> continuous
- joint RFinger32: limit lower=0 upper=0.86 effort=1 velocity=1 -> (none); type revolute -> continuous
- joint RFinger33: limit lower=0 upper=0.86 effort=1 velocity=1 -> (none); type revolute -> continuous
- joint RFinger41: limit lower=0 upper=0.86 effort=1 velocity=1 -> (none); type revolute -> continuous
- joint RFinger42: limit lower=0 upper=0.86 effort=1 velocity=1 -> (none); type revolute -> continuous
- joint RFinger43: limit lower=0 upper=0.86 effort=1 velocity=1 -> (none); type revolute -> continuous
- joint RShoulderPitch: origin xyz=-0.057 -0.14974 0.08682 rpy=0 0 0 -> xyz=-0.057 -0.14974 0.22582 rpy=0 0 0
- joint RThumb1: limit lower=0 upper=0.86 effort=1 velocity=1 -> (none); type revolute -> continuous
- joint RThumb2: limit lower=0 upper=0.86 effort=1 velocity=1 -> (none); type revolute -> continuous
- joint WheelB: axis 1.0 0 0 -> (none); limit lower=0 upper=0 effort=3.25 velocity=6.28319 -> (none)
- joint WheelFL: axis 1.0 0 0 -> (none); limit lower=0 upper=0 effort=3.25 velocity=6.28319 -> (none)
- joint WheelFR: axis 1.0 0 0 -> (none); limit lower=0 upper=0 effort=3.25 velocity=6.28319 -> (none)

File: urdf/pepper_ffb.urdf (robot description, URDF)
Before this commit: robot JulietteY20MP, 51 links, 50 joints
Links:
- added link CameraTop_frame
- added link CameraTop_optical_frame
- added link base_wheels_center
- added link rotz_link
- added link transx_link
- link Tibia: geometry collision mesh filename=package://pepper_description/meshes/KneePitch_0.10.stl scale=0.1 0.1 0.1; visual mesh filename=package://pepper_description/meshes/KneePitch.dae scale=0.1 0.1 0.1
- link WheelB_link: geometry collision mesh filename=package://pepper_description/meshes/WheelB_0.10.stl scale=0.1 0.1 0.1; visual mesh filename=package://pepper_description/meshes/WheelB.dae scale=0.1 0.1 0.1
- link WheelFL_link: geometry collision mesh filename=package://pepper_description/meshes/WheelFL_0.10.stl scale=0.1 0.1 0.1; visual mesh filename=package://pepper_description/meshes/WheelFL.dae scale=0.1 0.1 0.1
- link WheelFR_link: geometry collision mesh filename=package://pepper_description/meshes/WheelFR_0.10.stl scale=0.1 0.1 0.1; visual mesh filename=package://pepper_description/meshes/WheelFR.dae scale=0.1 0.1 0.1
Joints:
- removed joint base_footprint_joint
- removed joint base_link_fixedjoint
- added joint CameraTop_optical_frame_fixedjoint: type fixed, parent CameraTop_frame, child CameraTop_optical_frame, origin xyz=0 0 0 rpy=-1.57079632679 0 -1.57079632679
- added joint CameraTop_sensor_fixedjoint: type fixed, parent Head, child CameraTop_frame, origin xyz=0.08601 0 0.16284 rpy=0 0 0, axis 0 0 0
- added joint WheelB: type fixed, parent Tibia, child WheelB_link, origin xyz=-0.17 0 -0.264 rpy=0 0 -3.14159
- added joint WheelFL: type fixed, parent Tibia, child WheelFL_link, origin xyz=0.09 0.155 -0.264 rpy=0 0 1.07517
- added joint WheelFR: type fixed, parent Tibia, child WheelFR_link, origin xyz=0.09 -0.155 -0.264 rpy=0 0 -1.07517
- added joint leg_joint: type fixed, parent Tibia, child base_footprint, origin xyz=0. 0. -0.334 rpy=0 0 0
- added joint wheels_center_offset_joint: type fixed, parent base_footprint, child base_wheels_center, origin xyz=0.0062 0. 0. rpy=0 0 0
- joint HipPitch: axis 0 1.0 0 -> 0 -1.0 0
- joint KneePitch: axis 0 1.0 0 -> 0 -1.0 0
- joint Rot_Z: limit lower=0 upper=0 effort=3.25 velocity=6.28319 -> lower=0 upper=0 effort=5.0 velocity=0.5; origin xyz=0.0 0. 0. rpy=0 0 0 -> xyz=0.0 0. 0.334 rpy=0 0 0; parent WheelFL_link -> rotz_link
- joint Trans_X: child WheelFL_link -> rotz_link; limit lower=-10 upper=10 effort=3.25 velocity=6.28319 -> lower=-10 upper=10 effort=8.4 velocity=0.35; parent WheelB_link -> transx_link
- joint Trans_Y: child WheelB_link -> transx_link; limit lower=-10 upper=10 effort=3.25 velocity=6.28319 -> lower=-10 upper=10 effort=8.4 velocity=0.35; parent WheelFR_link -> base_link

Commit message: Added realsense (Pepper prototype)

File: urdf/pepper.urdf (robot description, URDF)
Before this commit: robot JulietteY20MP, 52 links, 51 joints
Links:
- added link RealSence_color_frame
- added link RealSence_color_optical_frame
- added link RealSence_depth_frame
- added link RealSence_depth_optical_frame
- added link RealSense_screw_frame; visual mesh filename=package://pepper_description/meshes/d435.dae
Joints:
- added joint RealSense_color_fixedjoint: type fixed, parent RealSense_screw_frame, child RealSence_color_frame, origin xyz=0 0.0325 0.0125 rpy=0 0 0
- added joint RealSense_color_optical_frame_fixedjoint: type fixed, parent RealSence_color_frame, child RealSence_color_optical_frame, origin xyz=0 0 0 rpy=-1.570796 0 -1.570796
- added joint RealSense_depth_fixedjoint: type fixed, parent RealSense_screw_frame, child RealSence_depth_frame, origin xyz=0 0.0175 0.0125 rpy=0 0 0
- added joint RealSense_depth_optical_frame_fixedjoint: type fixed, parent RealSence_depth_frame, child RealSence_depth_optical_frame, origin xyz=0 0 0 rpy=-1.570796 0 -1.570796
- added joint RealSense_fixedjoint: type fixed, parent CameraTop_frame, child RealSense_screw_frame, origin xyz=0.0 0.0 0.017 rpy=0 0 0, axis 0 0 0
- joint HeadPitch: limit lower=-0.706858 upper=0.637045 effort=2.666 velocity=9.22756 -> lower=-0.706858 upper=0.57 effort=2.666 velocity=9.22756
- joint HipRoll: axis 1.0 0 0 -> -1.0 0 0

Commit message: Description package clean up, update, adaptation for changes in robot module

File: urdf/pepper.urdf (robot description, URDF)
Before this commit: robot JulietteY20MP, 57 links, 56 joints
Links:
- added link camera_base; visual mesh filename=package://pepper_description/meshes/camera_base.stl
- added link camera_body; visual mesh filename=package://pepper_description/meshes/camera_body.stl
- added link camera_visor; visual mesh filename=package://pepper_description/meshes/camera_visor.stl
- added link kinect_depth_optical_frame
- added link kinect_imu_frame
- added link t265; visual mesh filename=package://pepper_description/meshes/t265.stl
- added link t265_pose
Joints:
- added joint camera_base_to_body: type fixed, parent camera_base, child camera_body, origin xyz=-0.0757 0. 0.008 rpy=0. 0. 0.
- added joint camera_base_to_visor: type fixed, parent camera_base, child camera_visor, origin xyz=0. 0. 0. rpy=0. 0. 0.
- added joint camera_realsense_to_azure: type fixed, parent RealSense_screw_frame, child camera_base, origin xyz=0.015 0.0005 0.045 rpy=0. 0. 0.
- added joint d435_to_t265: type fixed, parent RealSense_screw_frame, child t265, origin xyz=0. 0. 0.064 rpy=0. 0. 0.
- added joint kinect_depth_fixedjoint: type fixed, parent camera_base, child kinect_depth_optical_frame, origin xyz=0. 0. 0.0018 rpy=-1.675 0 -1.57
- added joint kinect_imu_fixedjoint: type fixed, parent camera_base, child kinect_imu_frame, origin xyz=-0.051074 -0.0033404 0.0027 rpy=3.14 0. 3.14
- added joint t265_pose_frame_joint: type fixed, parent t265, child t265_pose, origin xyz=0.00625 0.0 0.01225 rpy=0.0 0.0 0.0
- joint HeadPitch: limit lower=-0.706858 upper=0.57 effort=2.666 velocity=9.22756 -> lower=-0.706858 upper=0.43 effort=2.666 velocity=9.22756
- joint LHand: limit lower=0.02 upper=0.98 effort=0.144 velocity=12.56 -> lower=0 upper=1 effort=0.144 velocity=12.56
- joint RHand: limit lower=0.02 upper=0.98 effort=0.144 velocity=12.56 -> lower=0 upper=1 effort=0.144 velocity=12.56

Commit message: Added tablet frame

File: urdf/pepper.urdf (robot description, URDF)
Before this commit: robot JulietteY20MP, 64 links, 63 joints
Links:
- added link tablet
Joints:
- added joint tablet_fixedjoint: type fixed, parent torso, child tablet, origin xyz=0.0839249 0 0.2 rpy=0 -0.523599 0, axis 0 0 0

Commit message: [mesh] Extra camera mash updates

File: urdf/pepper.urdf (robot description, URDF)
Before this commit: robot JulietteY20MP, 65 links, 64 joints
Links:
- link RealSense_screw_frame: geometry visual mesh filename=package://pepper_description/meshes/d435.stl

Commit message: [mesh] Revert dae->stl mesh change

File: urdf/pepper.urdf (robot description, URDF)
Before this commit: robot JulietteY20MP, 65 links, 64 joints
Links:
- link RealSense_screw_frame: geometry visual mesh filename=package://pepper_description/meshes/d435.dae
